Commit message: 优化步态奖励

File: src/mjlab/asset_zoo/robots/custom_biped/urdf/biped.urdf (robot description, URDF)
Before this commit: robot biped, 7 links, 6 joints
Links:
- link left_ankle_link: mass 0.1529662 -> 0.1646342
- link left_knee_link: mass 0.4818865 -> 0.4824456
- link left_leg_Link: mass 0.6457834 -> 0.6942103
Joints:
- joint left_ankle_joint: origin xyz=0 -0.210703070258476 0.0153699569690486 rpy=0 0 0 -> xyz=0 -0.210003471144268 0.0145 rpy=0 0 0
- joint left_knee_joint: origin xyz=0.029996948741295 -0.22733201647225 -0.0538699569690269 rpy=0 0 0 -> xyz=0.0299965383151033 -0.228031615586488 -0.0529999999999996 rpy=0 0 0
- joint left_leg_joint: origin xyz=0 0.0633999999999999 -0.0300000000000169 rpy=1.5707963267949 0 0 -> xyz=0 0.0634000000000001 -0.0299999999999865 rpy=1.5707963267949 0 0
